File: converter.sch (KiCad schematic (older format))
At the start: 47 parts, among them J1 A04, J2 ???, J3 A01, J4 A02, J5 A03, J6 TEENSY INTERNAL PINS, J7 Screw_Terminal_01x02, J8 BLUEFRUIT LE SPI FRIEND, K1 DIP05-1C90-51D, U1 SSTW003A0A41Z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

Commit message: removing plots
Parts:
- added R1, R2: 100, Resistors_THT:R_Axial_DIN0204_L3.6mm_D1.6mm_P5.08mm_Vertical, symbol Device:R_Small_US
- J10: renamed from J?; value ??? -> B08
- J2: value ??? -> B08
- gave numbers to parts that had none: 33
Connections:
- net +5VD: now also U1.6 (VOUT+)
- net -48V: now also R1.2; no longer U1.2 (VIN-), U1.3 (~OFF)
- net GNDD: now also U1.4 (VOUT-)
- net RESTORE_MAGS: now also R2.2; no longer K1.2
- new net: K1.2, R2.1
- new net -VIN: R1.1, U1.2 (VIN-), U1.3 (~OFF)
Other:
- note added: "B08 : SECOND FRONT PANEL CONNECTOR\nA01 : FRONT PANEL CONNECTOR\nA02-A04 : KEYBOARD PANEL CONNECTORS"
- note removed: "??? : UNKOWN POSITION FRONT PANEL CONNECTOR\nA01 : FRONT PANEL CONNECTOR\nA02-A04 : KEYBOARD PANEL CONNECTORS"
- moved on the sheet: J7
